Commit message: 优化三机器人场景、全向底盘、避障与任务区域调度

File: src/hetero_fleet_description/urdf/heavy_diff_amr.xacro (robot description, xacro)
@@ -1,16 +1,8 @@
 <?xml version="1.0"?>
-<!-- Heavy differential-drive AMR for pallet transport.
-     SCALE: like the other two robots this is the warehouse design times `s`,
-     which is 0.45 here - NOT the 0.53 that MAP_SWAP.md's table still quotes.
-     The code is the source of truth: s=0.31 gives a 0.409 x 0.267 m body
-     (0.428 x 0.322 m including the bumper, wheels included), and the
-     controller geometry in heavy_diff_amr_controllers.yaml (wheel_radius
-     0.062 / separation 0.2945) was derived from exactly that. It started at
-     0.45 and has been shrunk twice since (0.36, now 0.31); see the note in
-     light_diff_amr.xacro. Masses scale as s^3, inertias as s^5, and the
-     shell mesh by s, so geometry, dynamics and visuals stay consistent.
-     The navigation footprint in robot_profiles.yaml (0.428 x 0.322 m) is
-     this same outline, measured by tools/measure_footprint.py.
--->
+<!-- Scene update 2026-10-10: all linear dimensions are twice the
+     previous model, scale s=0.62. Measured ground outline: 0.8556 × 0.6448 m.
+     Visual meshes, collision shapes, wheel positions and sensors share s;
+     masses scale with s^3 and inertias with s^5.
+     Controllers and Nav2 footprints must match this geometry. -->
 <robot xmlns:xacro="http://www.ros.org/wiki/xacro" name="heavy_diff_amr">
   <xacro:arg name="robot_name" default="heavy_1"/>
@@ -19,5 +11,5 @@
   <xacro:property name="controllers_file" value="$(arg controllers_file)"/>
   <xacro:property name="robot_name" value="$(arg robot_name)"/>
-  <xacro:property name="s" value="0.31"/>
+  <xacro:property name="s" value="0.62"/>
   <xacro:property name="base_length" value="${1.32 * s}"/>
   <xacro:property name="base_width" value="${0.86 * s}"/>

File: src/hetero_fleet_description/urdf/light_diff_amr.xacro (robot description, xacro)
@@ -1,19 +1,8 @@
 <?xml version="1.0"?>
-<!-- Lightweight differential-drive AMR, sized for the scanned office map.
-     SCALE: every dimension below is the warehouse design multiplied by `s`,
-     which is 0.60 here - NOT the 0.70 that MAP_SWAP.md's table still quotes.
-     The code is the source of truth: s=0.41 gives a 0.328 x 0.221 m body
-     (0.344 x 0.271 m including the bumper, wheels included), which is what
-     the controller geometry (wheel_radius 0.0451 / separation 0.246) and
-     tools/measure_footprint.py report. It started at 0.60 and has been
-     shrunk twice since (0.48, now 0.41): the ring corridor's narrowest
-     usable passage is ~1.1 m and every centimetre of robot width is
-     lateral room the controller gets to work with (see MAP_SWAP.md 3). Masses scale with volume (s^3)
-     and inertias with s^5, so the dynamics stay self-consistent; the shell
-     mesh is scaled by the same factor so the visuals match the collision
-     geometry.
-     The navigation footprint in robot_profiles.yaml (0.344 x 0.271 m) is
-     this same outline, measured by tools/measure_footprint.py.
--->
+<!-- Scene update 2026-10-10: all linear dimensions are twice the
+     previous model, scale s=0.82. Measured ground outline: 0.6888 × 0.5412 m.
+     Visual meshes, collision shapes, wheel positions and sensors share s;
+     masses scale with s^3 and inertias with s^5.
+     Controllers and Nav2 footprints must match this geometry. -->
 <robot xmlns:xacro="http://www.ros.org/wiki/xacro" name="light_diff_amr">
   <xacro:arg name="robot_name" default="light_1"/>
@@ -22,5 +11,5 @@
   <xacro:property name="controllers_file" value="$(arg controllers_file)"/>
   <xacro:property name="robot_name" value="$(arg robot_name)"/>
-  <xacro:property name="s" value="0.41"/>
+  <xacro:property name="s" value="0.82"/>
   <xacro:property name="base_length" value="${0.80 * s}"/>
   <xacro:property name="base_width" value="${0.54 * s}"/>

File: src/hetero_fleet_description/urdf/omni_mecanum_amr.xacro (robot description, xacro)
@@ -1,16 +1,6 @@
 <?xml version="1.0"?>
-<!-- Mecanum AMR for precise lateral docking.
-     SCALE: the warehouse design times `s`, which is 0.42 here. The code is the
-     source of truth: s=0.42 gives a 0.378 x 0.294 m body (0.403 x 0.353 m
-     including the bumper, wheels included), and the controller geometry in
-     omni_mecanum_amr_controllers.yaml (wheels_radius 0.0399, wheel joints at
-     x = +/-0.147, y = +/-0.1617) was derived from exactly that. It started at
-     0.61 and has been shrunk twice since (0.49, now 0.42); see the note in
-     light_diff_amr.xacro. Masses scale as s^3, inertias as s^5, the shell
-     mesh by s. The mecanum friction model - which is what makes this robot the
-     only one that can strafe - is unchanged; only its dimensions move.
-     The navigation footprint in robot_profiles.yaml (0.403 x 0.353 m) is
-     this same outline, measured by tools/measure_footprint.py.
--->
+<!-- Omni chassis update: s=0.70 (16.7% smaller than s=0.84), lower deck.
+     True footprint 0.672 x 0.588 m. Controller wheel geometry matches s.
+     Body inertia is computed from the actual box dimensions. -->
 <robot xmlns:xacro="http://www.ros.org/wiki/xacro" name="omni_mecanum_amr">
   <xacro:arg name="robot_name" default="omni_1"/>
@@ -19,13 +9,13 @@
   <xacro:property name="controllers_file" value="$(arg controllers_file)"/>
   <xacro:property name="robot_name" value="$(arg robot_name)"/>
-  <xacro:property name="s" value="0.42"/>
+  <xacro:property name="s" value="0.70"/>
   <xacro:property name="base_length" value="${0.90 * s}"/>
   <xacro:property name="base_width" value="${0.70 * s}"/>
-  <xacro:property name="base_height" value="${0.24 * s}"/>
+  <xacro:property name="base_height" value="${0.20 * s}"/>
   <xacro:property name="wheel_radius" value="${0.095 * s}"/>
   <xacro:property name="wheel_width" value="${0.070 * s}"/>
   <link name="base_footprint"/>
   <link name="base_link">
-    <inertial><mass value="${42.0 * s**3}"/><inertia ixx="${1.75 * s**5}" ixy="0" ixz="0" iyy="${2.25 * s**5}" iyz="0" izz="${3.10 * s**5}"/></inertial>
+    <inertial><origin xyz="0 0 ${base_height / 2}"/><mass value="${42.0 * s**3}"/><inertia ixx="${42.0 * s**3 * (base_width**2 + base_height**2) / 12}" ixy="0" ixz="0" iyy="${42.0 * s**3 * (base_length**2 + base_height**2) / 12}" iyz="0" izz="${42.0 * s**3 * (base_length**2 + base_width**2) / 12}"/></inertial>
     <visual><origin xyz="0 0 0"/><geometry><mesh filename="package://hetero_fleet_description/meshes/omni_shell.stl" scale="${s} ${s} ${s}"/></geometry><material name="red"><color rgba="0.78 0.10 0.12 1"/></material></visual>
     <collision><origin xyz="0 0 ${base_height / 2}"/><geometry><box size="${base_length} ${base_width} ${base_height}"/></geometry></collision>
@@ -46,21 +36,46 @@
   <link name="rear_right_corner_guard"><visual><origin xyz="0 0 ${0.12 * s}"/><geometry><cylinder radius="${0.05 * s}" length="${0.24 * s}"/></geometry><material name="guard"><color rgba="0.08 0.09 0.10 1"/></material></visual><collision><origin xyz="0 0 ${0.12 * s}"/><geometry><cylinder radius="${0.05 * s}" length="${0.24 * s}"/></geometry></collision></link>
   <joint name="rear_right_corner_guard_joint" type="fixed"><parent link="base_link"/><child link="rear_right_corner_guard"/><origin xyz="${-0.39 * s} ${-0.29 * s} 0"/></joint>
-  <xacro:macro name="mecanum_wheel" params="name x y">
+  <!-- X-arranged roller visuals; four smooth wheel collisions use the equivalent
+       free-roller constraints supplied by MecanumContacts in chassis coordinates. -->
+  <xacro:macro name="mecanum_roller" params="wheel index hand">
+    <xacro:property name="theta" value="${2*pi*index/16}"/>
+    <xacro:property name="axis_x" value="${hand*cos(theta)/sqrt(2)}"/>
+    <xacro:property name="axis_z" value="${-hand*sin(theta)/sqrt(2)}"/>
+    <link name="${wheel}_roller_${index}">
+      <visual><geometry><mesh filename="package://hetero_fleet_description/meshes/mecanum_barrel.stl"/></geometry><material name="roller"><color rgba="0.12 0.13 0.15 1"/></material></visual>
+    </link>
+    <joint name="${wheel}_roller_${index}_joint" type="fixed">
+      <parent link="${wheel}_wheel_link"/><child link="${wheel}_roller_${index}"/>
+      <origin xyz="${0.057*sin(theta)} 0 ${0.057*cos(theta)}" rpy="0 ${acos(axis_z)} ${atan2(1/sqrt(2),axis_x)}"/>
+    </joint>
+  </xacro:macro>
+  <xacro:macro name="mecanum_wheel" params="name x y hand">
     <link name="${name}_wheel_link">
-      <inertial><mass value="${0.65 * s**3}"/><inertia ixx="${0.004 * s**5}" ixy="0" ixz="0" iyy="${0.002 * s**5}" iyz="0" izz="${0.004 * s**5}"/></inertial>
-      <visual><origin rpy="${pi / 2} 0 0"/><geometry><cylinder radius="${wheel_radius}" length="${wheel_width}"/></geometry><material name="rubber"><color rgba="0.04 0.04 0.04 1"/></material></visual>
-      <!-- Keep this a cylinder, matching the visual. Replacing it with a
-           sphere was tried and is distinctly worse: with a point contact the
-           45 degree roller direction has nothing to push against and the
-           mecanum coupling disappears entirely - every command, strafe and
-           spin included, came out as straight-line +x motion. -->
-      <collision><origin rpy="${pi / 2} 0 0"/><geometry><cylinder radius="${wheel_radius}" length="${wheel_width}"/></geometry></collision>
+      <inertial><mass value="0.14"/><inertia ixx="${0.14*(3*0.035**2+wheel_width**2)/12}" ixy="0" ixz="0" iyy="${0.14*0.035**2/2}" iyz="0" izz="${0.14*(3*0.035**2+wheel_width**2)/12}"/></inertial>
+      <visual><origin rpy="${pi/2} 0 0"/><geometry><cylinder radius="0.045" length="${wheel_width}"/></geometry><material name="hub"><color rgba="0.04 0.04 0.04 1"/></material></visual>
+      <collision><origin rpy="${pi/2} 0 0"/><geometry><cylinder radius="${wheel_radius}" length="${wheel_width}"/></geometry></collision>
     </link>
-    <joint name="${name}_wheel_joint" type="continuous"><parent link="base_link"/><child link="${name}_wheel_link"/><origin xyz="${x} ${y} 0"/><axis xyz="0 1 0"/><limit effort="15" velocity="18"/></joint>
+    <joint name="${name}_wheel_joint" type="continuous"><parent link="base_link"/><child link="${name}_wheel_link"/><origin xyz="${x} ${y} 0"/><axis xyz="0 1 0"/><dynamics damping="0.002" friction="0"/><limit effort="15" velocity="18"/></joint>
+    <xacro:mecanum_roller wheel="${name}" index="0" hand="${hand}"/>
+    <xacro:mecanum_roller wheel="${name}" index="1" hand="${hand}"/>
+    <xacro:mecanum_roller wheel="${name}" index="2" hand="${hand}"/>
+    <xacro:mecanum_roller wheel="${name}" index="3" hand="${hand}"/>
+    <xacro:mecanum_roller wheel="${name}" index="4" hand="${hand}"/>
+    <xacro:mecanum_roller wheel="${name}" index="5" hand="${hand}"/>
+    <xacro:mecanum_roller wheel="${name}" index="6" hand="${hand}"/>
+    <xacro:mecanum_roller wheel="${name}" index="7" hand="${hand}"/>
+    <xacro:mecanum_roller wheel="${name}" index="8" hand="${hand}"/>
+    <xacro:mecanum_roller wheel="${name}" index="9" hand="${hand}"/>
+    <xacro:mecanum_roller wheel="${name}" index="10" hand="${hand}"/>
+    <xacro:mecanum_roller wheel="${name}" index="11" hand="${hand}"/>
+    <xacro:mecanum_roller wheel="${name}" index="12" hand="${hand}"/>
+    <xacro:mecanum_roller wheel="${name}" index="13" hand="${hand}"/>
+    <xacro:mecanum_roller wheel="${name}" index="14" hand="${hand}"/>
+    <xacro:mecanum_roller wheel="${name}" index="15" hand="${hand}"/>
   </xacro:macro>
-  <xacro:mecanum_wheel name="front_left" x="${base_length / 2 - 0.10 * s}" y="${base_width / 2 + wheel_width / 2}"/>
-  <xacro:mecanum_wheel name="front_right" x="${base_length / 2 - 0.10 * s}" y="${-base_width / 2 - wheel_width / 2}"/>
-  <xacro:mecanum_wheel name="rear_left" x="${-base_length / 2 + 0.10 * s}" y="${base_width / 2 + wheel_width / 2}"/>
-  <xacro:mecanum_wheel name="rear_right" x="${-base_length / 2 + 0.10 * s}" y="${-base_width / 2 - wheel_width / 2}"/>
+  <xacro:mecanum_wheel name="front_left" x="${base_length/2-0.10*s}" y="${base_width/2+wheel_width/2}" hand="1"/>
+  <xacro:mecanum_wheel name="front_right" x="${base_length/2-0.10*s}" y="${-base_width/2-wheel_width/2}" hand="-1"/>
+  <xacro:mecanum_wheel name="rear_left" x="${-base_length/2+0.10*s}" y="${base_width/2+wheel_width/2}" hand="-1"/>
+  <xacro:mecanum_wheel name="rear_right" x="${-base_length/2+0.10*s}" y="${-base_width/2-wheel_width/2}" hand="1"/>
   <link name="lidar_link">
     <inertial><mass value="0.15"/><inertia ixx="0.0002" ixy="0" ixz="0" iyy="0.0002" iyz="0" izz="0.0003"/></inertial>
@@ -74,48 +89,9 @@
   <gazebo reference="lidar_link"><sensor name="${robot_name}_lidar" type="gpu_lidar"><always_on>1</always_on><visualize>false</visualize><update_rate>20</update_rate><topic>/${robot_name}/scan</topic><frame_id>lidar_link</frame_id><lidar><scan><horizontal><samples>1080</samples><resolution>1</resolution><min_angle>-3.14159</min_angle><max_angle>3.14159</max_angle></horizontal></scan><range><min>0.10</min><max>15.0</max><resolution>0.01</resolution></range></lidar></sensor></gazebo>
   <xacro:fleet_gazebo_material link="base_link" rgba="0.78 0.10 0.12 1"/>
-  <!-- Mecanum wheels, modelled the way the rollers actually work.
-       Each roller spins freely about its own axis, and those axes lie at 45
-       degrees to the wheel plane - mirrored between the left and right sides.
-       So the *free sliding* direction is that 45 degree diagonal: fdir1 is
-       aligned with it and carries the low coefficient (mu1), while the
-       perpendicular diagonal grips (mu2). Getting this wrong (or leaving
-       fdir1 unset, when the engine picks the tangent directions itself) turns
-       the robot into something that can only ever slide forward: it cannot
-       strafe and it cannot even spin in place. -->
-  <!-- fdir1 lives in the *collision* frame, and the wheel collision is the
-       cylinder rotated by rpy = (+90, 0, 0): collision x is body x, but
-       collision z is body -y. The body-horizontal 45 degree diagonals
-       (1, +-1, 0)_body therefore read (1, 0, -+1) here. -->
-  <!-- Roller orientation. The left pair and the right pair carry opposite
-       diagonals; that mirroring is what lets a mecanum base strafe.
-       WHICH diagonal belongs on which side is not cosmetic, and the answer
-       here comes from measuring all three axes with tools/omni_probe.py
-       (twist published straight to the controller's reference topic, ground
-       truth read back from the odometry relay):
-         handedness        vx     wz                vy
-         left -1 right +1  1.00   -1.71  (INVERTED)  -0.14
-         left +1 right -1  0.98   +0.87 .. +0.97    -0.66 .. -1.30   <- this one
-       The previous revision used the first row. It looked fine because only
-       vx and the lateral magnitude were ever checked - but the plant turned
-       the OPPOSITE way to the command, at 1.7x the rate, so MPPI's
-       (DiffDrive) roll-outs predicted a turn the base never made: the
-       controller chased its own feedback, the robot snaked, and it could not
-       settle closer than ~0.35 m to a goal - which on a full run showed up as
-       omni_1 stalling 13 times where the other robots stalled 2-4, and as the
-       "navigation is a bit off" symptom on the vehicle.
-       The lateral sign is still mirrored: a +vy command moves the base -y,
-       which is why cmd_vel_stamper negates linear.y for this robot
-       (mirror_y). Both handednesses have that property, so mirror_y does not
-       depend on this choice. -->
-       mu1 runs along fdir1 and is the direction the rollers spin freely, so
-       it is kept deliberately small; mu2 grips across it and carries the
-       thrust, including the whole of a strafe. Tuning both was tried (0.02 /
-       1.0 -> 0.01 / 2.0) and changed the strafe response by under 1%, so the
-       original values are kept - the shortfall is not a friction tuning
-       problem. -->
-  <xacro:fleet_gazebo_wheel_dynamics link="front_left_wheel_link"  mu1="0.02" mu2="1.0" kp="100000" kd="1.0" fdir1="1 0 1"/>
-  <xacro:fleet_gazebo_wheel_dynamics link="rear_left_wheel_link"   mu1="0.02" mu2="1.0" kp="100000" kd="1.0" fdir1="1 0 1"/>
-  <xacro:fleet_gazebo_wheel_dynamics link="front_right_wheel_link" mu1="0.02" mu2="1.0" kp="100000" kd="1.0" fdir1="1 0 -1"/>
-  <xacro:fleet_gazebo_wheel_dynamics link="rear_right_wheel_link"  mu1="0.02" mu2="1.0" kp="100000" kd="1.0" fdir1="1 0 -1"/>
+  <gazebo><plugin filename="libhetero_mecanum_contacts.so" name="hetero_fleet::MecanumContacts"/></gazebo>
+  <xacro:fleet_gazebo_wheel_dynamics link="front_left_wheel_link" mu1="0.01" mu2="1.2" kp="100000" kd="20"/>
+  <xacro:fleet_gazebo_wheel_dynamics link="front_right_wheel_link" mu1="0.01" mu2="1.2" kp="100000" kd="20"/>
+  <xacro:fleet_gazebo_wheel_dynamics link="rear_left_wheel_link" mu1="0.01" mu2="1.2" kp="100000" kd="20"/>
+  <xacro:fleet_gazebo_wheel_dynamics link="rear_right_wheel_link" mu1="0.01" mu2="1.2" kp="100000" kd="20"/>
   <xacro:fleet_ros2_control name="${robot_name}" wheel_joints="${['front_left_wheel_joint', 'front_right_wheel_joint', 'rear_left_wheel_joint', 'rear_right_wheel_joint']}" controller_type="mecanum" controllers_file="${controllers_file}" namespace="${robot_name}"/>
 </robot>

Commit message: 保存狭窄项目源码及运行验证记录
Source: /home/ubuntu/huaxue304
Method: 贪心任务排程＋SIPP/PBS

File: src/hetero_fleet_description/urdf/heavy_diff_amr.xacro (robot description, xacro)
@@ -1,8 +1,4 @@
 <?xml version="1.0"?>
-<!-- Scene update 2026-10-10: all linear dimensions are twice the
-     previous model, scale s=0.62. Measured ground outline: 0.8556 × 0.6448 m.
-     Visual meshes, collision shapes, wheel positions and sensors share s;
-     masses scale with s^3 and inertias with s^5.
-     Controllers and Nav2 footprints must match this geometry. -->
+<!-- Reduced uniformly by 10% for fleet clearance; collision outline 1.4927886 x 1.125 m. -->
 <robot xmlns:xacro="http://www.ros.org/wiki/xacro" name="heavy_diff_amr">
   <xacro:arg name="robot_name" default="heavy_1"/>
@@ -11,5 +7,5 @@
   <xacro:property name="controllers_file" value="$(arg controllers_file)"/>
   <xacro:property name="robot_name" value="$(arg robot_name)"/>
-  <xacro:property name="s" value="0.62"/>
+  <xacro:property name="s" value="1.081730769210"/>
   <xacro:property name="base_length" value="${1.32 * s}"/>
   <xacro:property name="base_width" value="${0.86 * s}"/>

File: src/hetero_fleet_description/urdf/light_diff_amr.xacro (robot description, xacro)
@@ -1,8 +1,4 @@
 <?xml version="1.0"?>
-<!-- Scene update 2026-10-10: all linear dimensions are twice the
-     previous model, scale s=0.82. Measured ground outline: 0.6888 × 0.5412 m.
-     Visual meshes, collision shapes, wheel positions and sensors share s;
-     masses scale with s^3 and inertias with s^5.
-     Controllers and Nav2 footprints must match this geometry. -->
+<!-- Reduced uniformly by 10% for fleet clearance; collision outline 1.4318181 x 1.125 m. -->
 <robot xmlns:xacro="http://www.ros.org/wiki/xacro" name="light_diff_amr">
   <xacro:arg name="robot_name" default="light_1"/>
@@ -11,5 +7,5 @@
   <xacro:property name="controllers_file" value="$(arg controllers_file)"/>
   <xacro:property name="robot_name" value="$(arg robot_name)"/>
-  <xacro:property name="s" value="0.82"/>
+  <xacro:property name="s" value="1.704545454510"/>
   <xacro:property name="base_length" value="${0.80 * s}"/>
   <xacro:property name="base_width" value="${0.54 * s}"/>
@@ -55,5 +51,6 @@
       <collision><origin rpy="${pi / 2} 0 0"/><geometry><cylinder radius="${wheel_radius}" length="${wheel_width}"/></geometry></collision>
     </link>
-    <joint name="${side}_wheel_joint" type="continuous"><parent link="base_link"/><child link="${side}_wheel_link"/><origin xyz="0 ${y} 0"/><axis xyz="0 1 0"/><limit effort="8" velocity="18"/></joint>
+    <!-- Torque scales with mass times length; the body/inertia already use s^3/s^5. -->
+    <joint name="${side}_wheel_joint" type="continuous"><parent link="base_link"/><child link="${side}_wheel_link"/><origin xyz="0 ${y} 0"/><axis xyz="0 1 0"/><limit effort="${8 * s**4}" velocity="18"/></joint>
   </xacro:macro>
   <xacro:drive_wheel side="left" y="${base_width / 2 + wheel_width / 2}"/>

File: src/hetero_fleet_description/urdf/omni_mecanum_amr.xacro (robot description, xacro)
@@ -1,6 +1,4 @@
 <?xml version="1.0"?>
-<!-- Omni chassis update: s=0.70 (16.7% smaller than s=0.84), lower deck.
-     True footprint 0.672 x 0.588 m. Controller wheel geometry matches s.
-     Body inertia is computed from the actual box dimensions. -->
+<!-- Reduced uniformly by 10% for fleet clearance; collision outline 1.2857139 x 1.125 m. -->
 <robot xmlns:xacro="http://www.ros.org/wiki/xacro" name="omni_mecanum_amr">
   <xacro:arg name="robot_name" default="omni_1"/>
@@ -9,5 +7,5 @@
   <xacro:property name="controllers_file" value="$(arg controllers_file)"/>
   <xacro:property name="robot_name" value="$(arg robot_name)"/>
-  <xacro:property name="s" value="0.70"/>
+  <xacro:property name="s" value="1.339285714290"/>
   <xacro:property name="base_length" value="${0.90 * s}"/>
   <xacro:property name="base_width" value="${0.70 * s}"/>
